File: hardware/evse.kicad_pcb (KiCad board)
At the start: 2 copper layers, 42.5 x 62.5 mm, 85 parts, among them J101 Boot, P101 CON-SENSOR2, P102 Relay, P104 12V/Motor/GP, P105 CP/PP/PE, U101 XMC1100, U102 PEM1-S12-D12-S, U103 MAX14850, U104 ADS1118I, U105 OPA171AIDBV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

Commit message: fix bottom logo positions
Parts:
- moved G*** 2.18 mm to (160.2, 90.5)
- moved VAL 2.18 mm to (170.2, 90.5)
- moved VAL 2.18 mm to (150.2, 90.5)
Other:
- board text added: "Change Pin 2 + 3 for better PP resistor connection"
Changed lines of the file:
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@@
   (general
     (thickness 1.6)
-    (drawings 10)
+    (drawings 11)
     (tracks 1072)
     (zones 0)
@@
   )
   (layers
-    (0 F.Cu signal)
-    (31 B.Cu signal)
+    (0 F.Cu signal hide)
+    (31 B.Cu signal hide)
     (32 B.Adhes user)
     (33 F.Adhes user)
@@
     (aux_axis_origin 139 57.15)
     (grid_origin 139 57.15)
-    (visible_elements FFFEFFFF)
+    (visible_elements FFFFFFFF)
     (pcbplotparams
       (layerselection 0x010fc_ffffffff)
@@
   )
   (module kicad-libraries:Logo_CoMCU (layer B.Cu)
-    (at 160.2 88.35 180)
+    (at 160.2 90.525 180)
     (fp_text reference G*** (at 0 0) (layer B.SilkS) hide
       (effects (font (size 1.524 1.524) (thickness 0.3)) (justify mirror))
@@
   )
   (module kicad-libraries:WEEE_7mm (layer B.Cu)
-    (at 170.2 88.35 180)
+    (at 170.2 90.525 180)
     (fp_text reference VAL (at 0 0) (layer B.SilkS) hide
       (effects (font (size 0.2 0.2) (thickness 0.05)) (justify mirror))
@@
   )
   (module kicad-libraries:CE_5mm (layer B.Cu)
-    (at 150.2 88.35 180)
+    (at 150.2 90.525 180)
     (fp_text reference VAL (at 0 0) (layer B.SilkS) hide
       (effects (font (size 0.2 0.2) (thickness 0.05)) (justify mirror))
@@
     )
   )
+  (gr_text "Change Pin 2 + 3 for better PP resistor connection" (at 172.2 123.25) (layer F.Fab)
+    (effects (font (size 1 1) (thickness 0.15)))
+  )
   (gr_text tinkerforge.com (at 162.8 80.05) (layer F.SilkS)

Commit message: fixed typo
Other:
- board text added: "Charge"
- board text added: "Error"
- board text added: "Status"
- board text removed: "charge"
- board text removed: "error"
- board text removed: "status"
Changed lines of the file:
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@@
-(kicad_pcb (version 20171130) (host pcbnew 5.1.5-52549c5~84~ubuntu18.04.1)
+(kicad_pcb (version 20171130) (host pcbnew 5.1.5-52549c5~84~ubuntu19.04.1)
   (general
     (thickness 1.6)
@@
     (effects (font (size 0.8 0.8) (thickness 0.15)))
   )
-  (gr_text error (at 163.6 81.95) (layer F.SilkS)
+  (gr_text Error (at 163.6 81.95) (layer F.SilkS)
     (effects (font (size 0.75 0.75) (thickness 0.15)) (justify left))
   )
-  (gr_text charge (at 163.6 83.3) (layer F.SilkS)
+  (gr_text Charge (at 163.6 83.3) (layer F.SilkS)
     (effects (font (size 0.75 0.75) (thickness 0.15)) (justify left))
   )
-  (gr_text status (at 163.6 84.65) (layer F.SilkS)
+  (gr_text Status (at 163.6 84.65) (layer F.SilkS)
     (effects (font (size 0.75 0.75) (thickness 0.15)) (justify left))
   )

Commit message: changed cap value
Parts:
- Ce: renamed from C105; value 68uF/25V -> 100uF/35V
Changed lines of the file:
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@@
     (at 176.3 63.95 270)
     (attr smd)
-    (fp_text reference C105 (at 0 1.1 90) (layer F.Fab)
+    (fp_text reference Ce (at 0 1.1 90) (layer F.Fab)
       (effects (font (size 0.59944 0.59944) (thickness 0.12446)))
     )
-    (fp_text value 68uF/25V (at 0.95 -0.375 90) (layer F.Fab)
+    (fp_text value 100uF/35V (at 0.95 -0.375 90) (layer F.Fab)
       (effects (font (size 0.59944 0.59944) (thickness 0.12446)))
     )
