File: hardware/evse.kicad_pcb (KiCad board)
At the start: 2 copper layers, 42.5 x 62.5 mm, 87 parts, among them J101 Boot, P101 CON-SENSOR2, P102 Relay, P104 12V/Motor/GP, P105 CP/PP/PE, U101 XMC1100, U102 PEM1-S12-D12-S, U103 MAX14850, U104 ADS1118I, U105 OPA171AIDBV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

Commit message: small routing improvements
Routing:
- net RELAY: track 23.7 -> 25.7 mm
- net Net-(R114-Pad2): track 1.93 -> 3.85 mm
- net GND: track 92.1 -> 93.7 mm, vias 107 -> 108
Changed lines of the file:
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@@
     (thickness 1.6)
     (drawings 15)
-    (tracks 1121)
+    (tracks 1131)
     (zones 0)
     (modules 87)
@@
   (layers
     (0 F.Cu signal)
-    (31 B.Cu signal)
+    (31 B.Cu signal hide)
     (32 B.Adhes user)
     (33 F.Adhes user)
@@
   )
   (setup
-    (last_trace_width 0.3)
+    (last_trace_width 0.5)
     (user_trace_width 0.15)
     (user_trace_width 0.2)
@@
   (segment (start 158.75 77.25) (end 158.75 77.611092) (width 0.5) (layer F.Cu) (net 1))
   (segment (start 157.15 79.35) (end 157.15 79.1) (width 0.3) (layer F.Cu) (net 1))
-  (segment (start 158.475001 78.274999) (end 158.75 78) (width 0.3) (layer F.Cu) (net 1))
-  (segment (start 157.15 79.6) (end 158.475001 78.274999) (width 0.3) (layer F.Cu) (net 1))
   (segment (start 174 85.335) (end 174 85.05) (width 0.7) (layer F.Cu) (net 1))
   (segment (start 173.94375 85.39125) (end 174 85.335) (width 0.7) (layer F.Cu) (net 1))
@@
   (segment (start 160.325 76.75) (end 159.525 76.75) (width 0.3) (layer F.Cu) (net 1))
   (segment (start 159.025 77.25) (end 158.7 77.25) (width 0.3) (layer F.Cu) (net 1))
+  (segment (start 158.475001 78.274999) (end 158.75 78) (width 0.3) (layer F.Cu) (net 1))
+  (segment (start 157.775001 78.274999) (end 158.475001 78.274999) (width 0.3) (layer F.Cu) (net 1))
+  (segment (start 157.15 79.6) (end 157.15 78.9) (width 0.3) (layer F.Cu) (net 1))
+  (segment (start 157.15 78.9) (end 157.775001 78.274999) (width 0.3) (layer F.Cu) (net 1))
   (via (at 173.95 82.8) (size 0.55) (drill 0.25) (layers F.Cu B.Cu) (net 2))
   (segment (start 173.95 83.55) (end 173.95 82.8) (width 0.5) (layer F.Cu) (net 2))
@@
   (segment (start 160.325 76.25) (end 159.525 76.25) (width 0.3) (layer F.Cu) (net 2))
   (segment (start 159.025 75.75) (end 158.7 75.75) (width 0.3) (layer F.Cu) (net 2))
+  (segment (start 141.7 83) (end 142.5 83) (width 0.5) (layer F.Cu) (net 2))
+  (via (at 142.5 82.25) (size 0.55) (drill 0.25) (layers F.Cu B.Cu) (net 2))
+  (segment (start 142.5 83) (end 142.5 82.25) (width 0.5) (layer F.Cu) (net 2))
   (segment (start 176.45 106.8) (end 175.9 107.35) (width 0.3) (layer F.Cu) (net 3))
   (segment (start 177.2 106.8) (end 176.45 106.8) (width 0.3) (layer F.Cu) (net 3))
@@
   (segment (start 146.07 86.4) (end 146.07 85.1) (width 0.3) (layer F.Cu) (net 56))
   (segment (start 146.15 85.02) (end 146.15 84.5) (width 0.3) (layer F.Cu) (net 56))
+  (segment (start 146.07 86.4) (end 146.07 84.53) (width 0.5) (layer F.Cu) (net 56))
+  (segment (start 146.07 84.53) (end 146.1 84.5) (width 0.5) (layer F.Cu) (net 56))
   (via (at 145.05 83) (size 0.55) (drill 0.25) (layers F.Cu B.Cu) (net 57))
   (segment (start 145.05 83) (end 146.1 83) (width 0.25) (layer F.Cu) (net 57))
@@
   (segment (start 161.1 78.525) (end 161.1 79.1) (width 0.3) (layer F.Cu) (net 57))
   (segment (start 161.1 79.1) (end 161.05 79.15) (width 0.3) (layer F.Cu) (net 57))
+  (segment (start 146.1 83) (end 145.1 83) (width 0.5) (layer F.Cu) (net 57))
+  (segment (start 145.1 83) (end 145.05 83) (width 0.5) (layer F.Cu) (net 57))
+  (segment (start 145.05 83) (end 144.05 83) (width 0.5) (layer F.Cu) (net 57))
   (segment (start 160.11 94.36) (end 159.25 95.22) (width 0.7) (layer F.Cu) (net 59))
   (segment (start 159.25 95.22) (end 159.25 97.4) (width 0.7) (layer F.Cu) (net 59))
